File: DesigningMyFirstBadgeLife/LEDThrowie/LEDThrowie.kicad_pcb (KiCad board)
At the start: 2 copper layers, 43.4 x 43.4 mm, 7 parts

Commit message: Added section on exporting Gerbers.  Final part of #3
Routing:
- added copper zone on B.Cu, net GND
Changed lines of the file:
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@@
   (segment (start 136.511 96.52) (end 136.652 96.661) (width 0.25) (layer F.Cu) (net 3))
   (segment (start 120.396 96.52) (end 136.511 96.52) (width 0.25) (layer F.Cu) (net 3))
+  (zone (net 1) (net_name GND) (layer B.Cu) (hatch edge 0.508)
+    (connect_pads (clearance 0.508))
+    (min_thickness 0.254)
+    (fill yes (arc_segments 32) (thermal_gap 0.508) (thermal_bridge_width 0.508))
+    (polygon
+      (pts
+        (xy 151.384 107.696) (xy 102.87 107.696) (xy 102.87 62.992) (xy 151.13 62.992)
+      )
+    )
+  )
 )
